Commit message: Working initial simulation and navigation (chassis wheels and lasers)

File: robots/archie_mw/archie_mw.urdf.xacro (robot description, xacro)
@@ -1,5 +1,4 @@
 <?xml version="1.0" ?>
 <robot name="archie_mw" xmlns:xacro="http://www.ros.org/wiki/xacro">
-<!-- ####### GITHUB UPLOAD TEST############# -->
   <!-- PROPERTIES -->
   <xacro:include filename="$(find archie_simulation)/robots/archie_mw/xacros/properties.xacro" />
@@ -10,8 +9,9 @@
   <!--GAZEBO REFERENCES -->
   <xacro:include filename="$(find archie_simulation)/robots/archie_mw/xacros/archie_mw_gazebo.xacro" />
+  <xacro:include filename="$(find archie_simulation)/robots/archie_mw/xacros/archie_mw_colors_gazebo.xacro" />
   <!-- BODY -->
   <xacro:include filename="$(find archie_simulation)/robots/archie_mw/xacros/archie_mw_body.xacro" />
   <!-- WHEELS -->
-  <xacro:include filename="$(find archie_simulation)/robots/archie_mw/xacros/omni_wheel.xacro" />
+  <!-- <xacro:include filename="$(find archie_simulation)/robots/archie_mw/xacros/omni_wheel.xacro" /> -->
   <xacro:include filename="$(find archie_simulation)/robots/archie_mw/xacros/mecanum_wheel.xacro" />
   <!-- SENSORS -->
@@ -46,24 +46,24 @@
     width="${chassis_width}" height="${chassis_height}" mass="${chassis_weight}"
     color="Yellow" z_offset="${chassis_center_to_base_footprint_z_offset}">
-    <origin xyz="0 0 0" rpy="0 0 0" />
+    <joint_origin xyz="0 0 0" rpy="0 0 0" />
   </xacro:archie_mw_base>
 <!--  -->
   <!-- Wheel Macro -->
-  <xacro:mecanum_wheel_152 name="archie_mw_omni_wheel_front_left" parent="base_footprint" diameter="${wheel_diameter}" width="${wheel_width}" mass="${wheel_weight}" color="White"
+  <xacro:mecanum_wheel_152 name="archie_mw_mecanum_wheel_front_left" parent="base_footprint" diameter="${wheel_diameter}" width="${wheel_width}" mass="${wheel_weight}" color="White"
       mesh_file_name="package://archie_simulation/robots/archie_mw/meshes/mecanum_wheel_left.STL" mesh_scale_x="${1*SCALE_mm_to_m}"
       mesh_scale_y="${0.92*SCALE_mm_to_m}" mesh_scale_z="${1.52*SCALE_mm_to_m}">
     <origin xyz="${left_front_wheel_x_offset} ${left_front_wheel_y_offset+shaft_lenght} ${left_front_wheel_z_offset}" rpy="0 0 0" />
   </xacro:mecanum_wheel_152>
-  <xacro:mecanum_wheel_152 name="archie_mw_omni_wheel_front_right" parent="base_link" diameter="${wheel_diameter}" width="${wheel_width}" mass="${wheel_weight}" color="White"
+  <xacro:mecanum_wheel_152 name="archie_mw_mecanum_wheel_front_right" parent="base_link" diameter="${wheel_diameter}" width="${wheel_width}" mass="${wheel_weight}" color="White"
       mesh_file_name="package://archie_simulation/robots/archie_mw/meshes/mecanum_wheel_right.STL" mesh_scale_x="${1*SCALE_mm_to_m}"
       mesh_scale_y="${0.92*SCALE_mm_to_m}" mesh_scale_z="${1.52*SCALE_mm_to_m}">
     <origin xyz="${left_front_wheel_x_offset} ${-(left_front_wheel_y_offset+shaft_lenght)} ${left_front_wheel_z_offset}" rpy="0 0 0" />
   </xacro:mecanum_wheel_152>
-  <xacro:mecanum_wheel_152 name="archie_mw_omni_wheel_back_left" parent="base_link" diameter="${wheel_diameter}" width="${wheel_width}" mass="${wheel_weight}" color="White"
+  <xacro:mecanum_wheel_152 name="archie_mw_mecanum_wheel_back_left" parent="base_link" diameter="${wheel_diameter}" width="${wheel_width}" mass="${wheel_weight}" color="White"
       mesh_file_name="package://archie_simulation/robots/archie_mw/meshes/mecanum_wheel_left.STL" mesh_scale_x="${1*SCALE_mm_to_m}"
       mesh_scale_y="${0.92*SCALE_mm_to_m}" mesh_scale_z="${1.52*SCALE_mm_to_m}">
     <origin xyz="${-left_front_wheel_x_offset} ${left_front_wheel_y_offset+shaft_lenght} ${left_front_wheel_z_offset}" rpy="0 0 0" />
   </xacro:mecanum_wheel_152>
-  <xacro:mecanum_wheel_152 name="archie_mw_omni_wheel_back_right" parent="base_link" diameter="${wheel_diameter}" width="${wheel_width}" mass="${wheel_weight}" color="White"
+  <xacro:mecanum_wheel_152 name="archie_mw_mecanum_wheel_back_right" parent="base_link" diameter="${wheel_diameter}" width="${wheel_width}" mass="${wheel_weight}" color="White"
       mesh_file_name="package://archie_simulation/robots/archie_mw/meshes/mecanum_wheel_right.STL" mesh_scale_x="${1*SCALE_mm_to_m}"
       mesh_scale_y="${0.92*SCALE_mm_to_m}" mesh_scale_z="${1.52*SCALE_mm_to_m}">
@@ -72,14 +72,14 @@
 <!-- ####################### -->
 <!-- ${ROTATE_90_DEGREES} -->
-  <!-- <xacro:omni_wheel_250 name="archie_mw_omni_wheel_front_left" parent="base_footprint">
+  <!-- <xacro:omni_wheel_250 name="archie_mw_mecanum_wheel_front_left" parent="base_footprint">
     <origin xyz="0.25 0.28 0.13" rpy="0 0 0" />
   </xacro:omni_wheel_250>
-  <xacro:omni_wheel_250 name="archie_mw_omni_wheel_front_right" parent="base_footprint">
+  <xacro:omni_wheel_250 name="archie_mw_mecanum_wheel_front_right" parent="base_footprint">
     <origin xyz="0.25 -0.28 0.13" rpy="0 0 3.14" />
   </xacro:omni_wheel_250>
-  <xacro:omni_wheel_250 name="archie_mw_omni_wheel_back_left" parent="base_footprint">
+  <xacro:omni_wheel_250 name="archie_mw_mecanum_wheel_back_left" parent="base_footprint">
     <origin xyz="-0.25 0.28 0.13" rpy="0 0 0" />
   </xacro:omni_wheel_250>
-  <xacro:omni_wheel_250 name="archie_mw_omni_wheel_back_right" parent="base_footprint">
+  <xacro:omni_wheel_250 name="archie_mw_mecanum_wheel_back_right" parent="base_footprint">
     <origin xyz="-0.25 -0.28 0.13" rpy="0 0 3.14" />
   </xacro:omni_wheel_250> -->
@@ -170,37 +170,37 @@
     <origin xyz="0 0 0.38" rpy="0 0 0" />
   </xacro:camera> -->
-  <transmission name="archie_mw_omni_wheel_front_left">
-    <type>transmission_interface/SimpleTransmission</type>
-    <joint name="archie_mw_omni_wheel_front_left_joint">
-      <hardwareInterface>hardware_interface/VelocityJointInterface</hardwareInterface>
-    </joint>
-    <actuator name="archie_mw_omni_wheel_front_left_motor">
-      <mechanicalReduction>1</mechanicalReduction>
-    </actuator>
-  </transmission>
-  <transmission name="archie_mw_omni_wheel_front_right">
-    <type>transmission_interface/SimpleTransmission</type>
-    <joint name="archie_mw_omni_wheel_front_right_joint">
-      <hardwareInterface>hardware_interface/VelocityJointInterface</hardwareInterface>
-    </joint>
-    <actuator name="archie_mw_omni_wheel_front_right_motor">
-      <mechanicalReduction>1</mechanicalReduction>
-    </actuator>
-  </transmission>
-  <transmission name="archie_mw_omni_wheel_back_left">
-    <type>transmission_interface/SimpleTransmission</type>
-    <joint name="archie_mw_omni_wheel_back_left_joint">
-      <hardwareInterface>hardware_interface/VelocityJointInterface</hardwareInterface>
-    </joint>
-    <actuator name="archie_mw_omni_wheel_back_left_motor">
-      <mechanicalReduction>1</mechanicalReduction>
-    </actuator>
-  </transmission>
-  <transmission name="archie_mw_omni_wheel_back_right">
-    <type>transmission_interface/SimpleTransmission</type>
-    <joint name="archie_mw_omni_wheel_back_right_joint">
-      <hardwareInterface>hardware_interface/VelocityJointInterface</hardwareInterface>
-    </joint>
-    <actuator name="archie_mw_omni_wheel_back_right_motor">
+  <transmission name="archie_mw_mecanum_wheel_front_left">
+    <type>transmission_interface/SimpleTransmission</type>
+    <joint name="archie_mw_mecanum_wheel_front_left_joint">
+      <hardwareInterface>hardware_interface/VelocityJointInterface</hardwareInterface>
+    </joint>
+    <actuator name="archie_mw_mecanum_wheel_front_left_motor">
+      <mechanicalReduction>1</mechanicalReduction>
+    </actuator>
+  </transmission>
+  <transmission name="archie_mw_mecanum_wheel_front_right">
+    <type>transmission_interface/SimpleTransmission</type>
+    <joint name="archie_mw_mecanum_wheel_front_right_joint">
+      <hardwareInterface>hardware_interface/VelocityJointInterface</hardwareInterface>
+    </joint>
+    <actuator name="archie_mw_mecanum_wheel_front_right_motor">
+      <mechanicalReduction>1</mechanicalReduction>
+    </actuator>
+  </transmission>
+  <transmission name="archie_mw_mecanum_wheel_back_left">
+    <type>transmission_interface/SimpleTransmission</type>
+    <joint name="archie_mw_mecanum_wheel_back_left_joint">
+      <hardwareInterface>hardware_interface/VelocityJointInterface</hardwareInterface>
+    </joint>
+    <actuator name="archie_mw_mecanum_wheel_back_left_motor">
+      <mechanicalReduction>1</mechanicalReduction>
+    </actuator>
+  </transmission>
+  <transmission name="archie_mw_mecanum_wheel_back_right">
+    <type>transmission_interface/SimpleTransmission</type>
+    <joint name="archie_mw_mecanum_wheel_back_right_joint">
+      <hardwareInterface>hardware_interface/VelocityJointInterface</hardwareInterface>
+    </joint>
+    <actuator name="archie_mw_mecanum_wheel_back_right_motor">
       <mechanicalReduction>1</mechanicalReduction>
     </actuator>

File: robots/archie_mw/xacros/archie_mw_body.xacro (robot description, xacro)
@@ -1,7 +1,7 @@
 <?xml version="1.0"?>
 <robot xmlns:xacro="http://www.ros.org/wiki/xacro" name="archie_mw">
-  <xacro:macro name="archie_mw_base" params="name parent *origin lenght width height mass color z_offset">
+  <xacro:macro name="archie_mw_base" params="name parent *joint_origin lenght width height mass color z_offset">
     <joint name="${name}_joint" type="fixed">
-      <xacro:insert_block name="origin" />
+      <xacro:insert_block name="joint_origin" />
         <axis xyz="0 0 -1" />
       <!-- <limit effort="1000.0" lower="-1e+16" upper="1e+16" velocity="3.5"/> -->
@@ -29,11 +29,16 @@
         </geometry>
       </collision>
-    <inertial>
-      <mass value="${mass}" />
-      <origin xyz="0 0 ${z_offset}" rpy="0 0 0" />
-      <inertia ixx="${0.0833333 * mass * (width*width + height*height)}" ixy="0.0" ixz="0.0"
-        iyy="${0.0833333 * mass * (lenght*lenght + height*height)}" iyz="0.0"
-        izz="${0.0833333 * mass * (lenght*lenght + width*width)}" />
-    </inertial>
+      <inertial>
+        <mass value="${mass}" />
+        <origin xyz="0 0 ${z_offset}" rpy="0 0 0" />
+        <inertia ixx="${0.0833333 * mass * (width*width + height*height)}" ixy="0.0" ixz="0.0"
+          iyy="${0.0833333 * mass * (lenght*lenght + height*height)}" iyz="0.0"
+          izz="${0.0833333 * mass * (lenght*lenght + width*width)}" />
+      </inertial>
+      <!-- <inertial>
+        <xacro:box_inertial_with_origin x="${lenght}" y="${width}" z="${height}" mass="${mass}">
+          <origin xyz="0 0 ${z_offset}" rpy="0 0 0" />
+        </xacro:box_inertial_with_origin>
+      </inertial> -->
     </link>
   </xacro:macro>

File: robots/archie_mw/xacros/mecanum_wheel.xacro (robot description, xacro)
@@ -53,5 +53,5 @@
       <mu1>0.0001</mu1>
       <mu2>0.0001</mu2>
-    <material>Gazebo/Blue</material>
+    <material>Gazebo/Grey</material>
     </gazebo>
   </xacro:macro>

Commit message: Add electronics box on top of the chassis

File: robots/archie_mw/archie_mw.urdf.xacro (robot description, xacro)
@@ -48,6 +48,16 @@
     <joint_origin xyz="0 0 0" rpy="0 0 0" />
   </xacro:archie_mw_base>
-<!--  -->
-  <!-- Wheel Macro -->
+<!-- **** ELECTRONICS BOX (MODULE) - height 100 mm ****  -->
+<!-- /batteries height is 76 mm whenlaying on the side. -->
+<!-- can accomadete, not only Raspberry PI 4 with passive cooling case,  -->
+<!-- but also  Intel NUC in the big case 51 mm height/ -->
+<!-- ! The Joint is positioned on top plane of the chassis (base_link) module -->
+  <xacro:fixed_joint name="electronics_box" parent_name="base_footprint" child_name="electronics_box" color="Grey">
+    <origin xyz="0 0 ${(chassis_center_to_base_footprint_z_offset + chassis_half_height)}" rpy="0 0 0" />
+  </xacro:fixed_joint>
+  <xacro:box_link name="electronics_box" lenght="${electronics_box_lenght}" width="${electronics_box_width}" height="${electronics_box_height}" mass="${electronics_box_weight}" color="Light_grey">
+    <origin xyz="0 0 0" rpy="0 0 0" />
+  </xacro:box_link>
+  <!-- Invoke Wheel Macros -->
   <xacro:mecanum_wheel_152 name="archie_mw_mecanum_wheel_front_left" parent="base_footprint" diameter="${wheel_diameter}" width="${wheel_width}" mass="${wheel_weight}" color="White"
       mesh_file_name="package://archie_simulation/robots/archie_mw/meshes/mecanum_wheel_left.STL" mesh_scale_x="${1*SCALE_mm_to_m}"

File: robots/archie_mw/xacros/archie_mw_body.xacro (robot description, xacro)
@@ -43,3 +43,47 @@
     </link>
   </xacro:macro>
+    <!-- #### FIXED JOINT MACRO #### -->
+    <xacro:macro name="fixed_joint" params="name parent_name child_name color *origin">
+      <joint name="${name}_joint" type="fixed">
+        <parent link="${parent_name}"/>
+        <child link="${child_name}"/>
+        <xacro:insert_block name="origin" />
+      </joint>
+    </xacro:macro>
+      <!-- #### BOX MACRO #### -->
+    <xacro:macro name="box_link" params="name lenght width height mass color *origin">
+      <link name="${name}">
+        <visual>
+        <!-- The chassis is represented with a box and the origin of that box is in it's center.
+        That's why, in order to visualize properly, we need to add half of the box height to
+        the distance from the ground allready defined in the joint. -->
+          <origin xyz="0 0 ${height/2}" rpy="0 0 0" />
+          <geometry>
+            <!-- <mesh filename="package://archie_simulation/robots/archie_mw/meshes/archie_electronics_link.STL" scale="0.001 0.001 0.001"/> -->
+            <box size="${lenght} ${width} ${height}"/>
+          </geometry>
+          <!-- <material name="light_grey" /> -->
+          <material name="${color}" />
+        </visual>
+        <collision>
+          <origin xyz="0 0 0" rpy="0 0 0" />
+          <geometry>
+            <box size="${lenght} ${width} ${height}"/>
+          </geometry>
+        </collision>
+          <!-- Ivoke box_inertial_with_origin macro -->
+        <!-- <xacro:box_inertial_with_origin x="${lenght}" y="${width}" z="${height}" mass="${mass}">
+          <origin xyz="0 0 0" rpy="0 0 0" />
+        </xacro:box_inertial_with_origin> -->
+        <inertial>
+          <mass value="${mass}" />
+          <!-- <origin xyz="0 0 ${z_offset}" rpy="0 0 0" /> -->
+          <!-- ! Should we offset to the center of the box here??????????? -->
+          <origin xyz="0 0 0" rpy="0 0 0" />
+          <inertia ixx="${0.0833333 * mass * (width*width + height*height)}" ixy="0.0" ixz="0.0"
+            iyy="${0.0833333 * mass * (lenght*lenght + height*height)}" iyz="0.0"
+            izz="${0.0833333 * mass * (lenght*lenght + width*width)}" />
+        </inertial>
+      </link>
+    </xacro:macro>
 </robot>

File: robots/archie_mw/xacros/properties.xacro (robot description, xacro)
@@ -28,4 +28,10 @@
     <!-- <xacro:property name="chassis_center_to_base_footprint_z_offset" value="${86.2*SCALE_mm_to_m + chassis_half_height}" />  -->
     <xacro:property name="chassis_center_to_base_footprint_z_offset" value="${86.2*SCALE_mm_to_m}" />  <!--- From the ground to the middle of the chassis-->
+  <!-- ELECTRONICS BOX DIMENSIONS  -->
+    <xacro:property name="electronics_box_lenght" value="${chassis_lenght}" />
+    <xacro:property name="electronics_box_width" value="${chassis_width}" />
+    <xacro:property name="electronics_box_height" value="${100*SCALE_mm_to_m}" />
+    <xacro:property name="electronics_box_half_height" value="${electronics_box_height/2}" />
+    <xacro:property name="electronics_box_weight" value="${15}" /> <!-- in kg-->
     <!-- MOTOR WITH SUPPORT AND ELASTIC CLUTCH COUPLER DIMENSIONS  -->
     <!--  2.16 Kg - approximate with a box: h: 69 w: 60 l: 71+133.5+19 =223.5-->

Commit message: wip - change names

File: robots/archie_mw/archie_mw.urdf.xacro (robot description, xacro)
@@ -81,24 +81,12 @@
   </xacro:mecanum_wheel_152>
 <!-- ####################### -->
-<!-- ${ROTATE_90_DEGREES} -->
-  <!-- <xacro:omni_wheel_250 name="archie_mw_mecanum_wheel_front_left" parent="base_footprint">
-    <origin xyz="0.25 0.28 0.13" rpy="0 0 0" />
-  </xacro:omni_wheel_250>
-  <xacro:omni_wheel_250 name="archie_mw_mecanum_wheel_front_right" parent="base_footprint">
-    <origin xyz="0.25 -0.28 0.13" rpy="0 0 3.14" />
-  </xacro:omni_wheel_250>
-  <xacro:omni_wheel_250 name="archie_mw_mecanum_wheel_back_left" parent="base_footprint">
-    <origin xyz="-0.25 0.28 0.13" rpy="0 0 0" />
-  </xacro:omni_wheel_250>
-  <xacro:omni_wheel_250 name="archie_mw_mecanum_wheel_back_right" parent="base_footprint">
-    <origin xyz="-0.25 -0.28 0.13" rpy="0 0 3.14" />
-  </xacro:omni_wheel_250> -->
   <!-- Sensors -->
   <xacro:sick_laser_v0 name="lidar_1" parent="base_link" ros_topic="lidar_1/scan_filtered">
     <origin xyz="0.442 0 0.372" rpy="0 0 0" />
   </xacro:sick_laser_v0>
+<!--
   <xacro:sick_laser_v0 name="lidar_2" parent="base_link" ros_topic="lidar_2/scan_filtered">
     <origin xyz="-0.442 0 0.372" rpy="0 0 3.14" />
-  </xacro:sick_laser_v0>
+  </xacro:sick_laser_v0> -->
   <!--+++++++++++++++++++ IMU ++++++++++++++++++++++++-->
   <!-- Comment or uncomment based on your requirement -->
