Commit message: Add depth camera and docking adapter

File: robots/archie_mw/archie_mw.urdf.xacro (robot description, xacro)
@@ -15,4 +15,6 @@
   <!-- <xacro:include filename="$(find archie_simulation)/robots/archie_mw/xacros/omni_wheel.xacro" /> -->
   <xacro:include filename="$(find archie_simulation)/robots/archie_mw/xacros/mecanum_wheel.xacro" />
+  <!--DOCKING ADAPTER  -->
+  <xacro:include filename="$(find archie_simulation)/robots/archie_mw/xacros/docking_adapter.xacro" />
   <!-- SENSORS -->
   <!-- <xacro:include filename="$(find archie_simulation)/robots/archie_mw/xacros/sick_S300.xacro" /> -->
@@ -20,4 +22,6 @@
   <xacro:include filename="$(find archie_simulation)/robots/archie_mw/xacros/micro_scan.xacro" />
   <!--Ultrasonics, cameras and IMU's  -->
+  <!-- Depth Camera Realsense d435i-->
+  <xacro:include filename="$(find archie_simulation)/robots/archie_mw/xacros/depth_camera.xacro" />
   <!-->
   <xacro:include filename="$(find archie_simulation)/robots/archie_mw/xacros/imu.xacro" />
@@ -53,6 +57,8 @@
 <!-- but also  Intel NUC in the big case 51 mm height/ -->
 <!-- ! The Joint is positioned on top plane of the chassis (base_link) module -->
-  <xacro:fixed_joint name="electronics_box" parent_name="base_footprint" child_name="electronics_box" color="Grey">
-    <origin xyz="0 0 ${(chassis_center_to_base_footprint_z_offset + chassis_half_height)}" rpy="0 0 0" />
+  <!-- <xacro:fixed_joint name="electronics_box" parent_name="base_footprint" child_name="electronics_box" color="Grey">
+    <origin xyz="0 0 ${electronics_box_z_offset}" rpy="0 0 0" /> -->
+  <xacro:fixed_joint name="electronics_box" parent_name="base_link" child_name="electronics_box" color="Grey">
+    <origin xyz="0 0 ${130.7*SCALE_mm_to_m}" rpy="0 0 0" />
   </xacro:fixed_joint>
   <xacro:box_link name="electronics_box" lenght="${electronics_box_lenght}" width="${electronics_box_width}" height="${electronics_box_height}" mass="${electronics_box_weight}" color="Light_grey">
@@ -80,13 +86,28 @@
     <origin xyz="${-left_front_wheel_x_offset} ${-(left_front_wheel_y_offset+shaft_lenght)} ${left_front_wheel_z_offset}" rpy="0 0 0" />
   </xacro:mecanum_wheel_152>
+<!--Docking adapter Macro  -->
+  <xacro:docking_adapter name="docking_adapter" parent="base_link">
+    <origin xyz="-0.300 0 0.320" rpy="0 0 -1.57" />
+  </xacro:docking_adapter>
 <!-- ####################### -->
   <!-- Sensors -->
+  <xacro:fixed_joint name="rplidar_a2_laser_beam_joint" parent_name="electronics_box" child_name="rplidar_a2_laser_beam_link" color="Red">
+    <origin xyz="${rplidar_a2_laser_beam_joint_x_offset} ${rplidar_a2_laser_beam_joint_y_offset} ${electronics_box_height}" rpy="0 0 ${ROTATE_180_DEGREES}" />
+  </xacro:fixed_joint>
+  <xacro:box_link name="rplidar_a2_laser_beam_link" lenght="${0.041}" width="${0.041}" height="${0.001}" mass="${0.005}" color="Red">
+    <origin xyz="0 0 0" rpy="0 0 0" />
+  </xacro:box_link>
+  <!-- <xacro:fixed_joint name="rplidar_a2_laser_beam_fom_base_link_joint" parent_name="base_link" child_name="rplidar_a2_laser_beam_fom_base_link_link" color="Red">
+    <origin xyz="${rplidar_a2_laser_beam_joint_x_offset} ${rplidar_a2_laser_beam_joint_y_offset} ${230.7*SCALE_mm_to_m}" rpy="0 0 ${ROTATE_180_DEGREES}" />
+  </xacro:fixed_joint>
+  <xacro:box_link name="rplidar_a2_laser_beam_fom_base_link_link" lenght="${0.060}" width="${0.02}" height="${0.001}" mass="${0.005}" color="Green">
+    <origin xyz="0 0 0" rpy="0 0 0" />
+  </xacro:box_link> -->
   <xacro:sick_laser_v0 name="lidar_1" parent="base_link" ros_topic="lidar_1/scan_filtered">
     <origin xyz="0.442 0 0.372" rpy="0 0 0" />
   </xacro:sick_laser_v0>
-<!--
   <xacro:sick_laser_v0 name="lidar_2" parent="base_link" ros_topic="lidar_2/scan_filtered">
     <origin xyz="-0.442 0 0.372" rpy="0 0 3.14" />
-  </xacro:sick_laser_v0> -->
+  </xacro:sick_laser_v0>
   <!--+++++++++++++++++++ IMU ++++++++++++++++++++++++-->
   <!-- Comment or uncomment based on your requirement -->
@@ -168,4 +189,9 @@
     <origin xyz="0 0 0.38" rpy="0 0 0" />
   </xacro:camera> -->
+  <!-- Depth Camera -->
+  <xacro:depth_camera name="camera" parent="base_link">
+    <origin xyz="-0.228 0.015 0.461" rpy="0 0 3.14159" />
+  </xacro:depth_camera>
+  <!-- TRANSMISSIONS -->
   <transmission name="archie_mw_mecanum_wheel_front_left">
     <type>transmission_interface/SimpleTransmission</type>

File: robots/archie_mw/xacros/archie_mw_body.xacro (robot description, xacro)
@@ -4,5 +4,5 @@
     <joint name="${name}_joint" type="fixed">
       <xacro:insert_block name="joint_origin" />
-        <axis xyz="0 0 -1" />
+        <!-- <axis xyz="0 0 -1" />   remove this???????????? -->
       <!-- <limit effort="1000.0" lower="-1e+16" upper="1e+16" velocity="3.5"/> -->
       <joint_properties damping="1" friction="1" />

File: robots/archie_mw/xacros/archie_mw_gazebo.xacro (robot description, xacro)
@@ -1,4 +1,9 @@
 <?xml version="1.0"?>
 <robot name="archie_mw" xmlns:xacro="http://www.ros.org/wiki/xacro">
+<!-- TODO Is this gravity and self colide needed????????????????/ -->
+   <gazebo reference="base_link">
+    <gravity>true</gravity>
+    <self_collide>false</self_collide>
+  </gazebo>
   <!-- Lidar sensors -->
   <gazebo reference="lidar_1_link">
@@ -72,7 +77,59 @@
         </sensor>
   </gazebo>
-  <!-- Camera -->
+  <!-- Depth Camera -->
+  <gazebo reference="camera_link_gazebo">
+    <sensor name="camera1" type="depth">
+      <update_rate>15</update_rate>
+      <hfov>70</hfov>
+      <camera name="head">
+        <image>
+          <width>320</width>
+          <height>240</height>
+          <format>R8G8B8</format>
+        </image>
+        <clip>
+          <near>0.02</near>
+          <far>300</far>
+        </clip>
+        <noise>
+          <type>gaussian</type>
+          <!-- Noise is sampled independently per pixel on each frame.
+               That pixel's noise value is added to each of its color
+               channels, which at that point lie in the range [0,1]. -->
+          <mean>0.0</mean>
+          <stddev>0.03</stddev>
+        </noise>
+      </camera>
+      <plugin name="camera1_controller" filename="libgazebo_ros_openni_kinect.so">
+        <!--<baseline>0.2</baseline>-->
+        <alwaysOn>true</alwaysOn>
+        <updateRate>0.0</updateRate>
+        <cameraName>camera_ir</cameraName>
+        <imageTopicName>/camera/depth/image_raw</imageTopicName>
+        <cameraInfoTopicName>/camera/depth/camera_info</cameraInfoTopicName>
+        <depthImageTopicName>/camera/depth/depth_raw</depthImageTopicName>
+        <depthImageInfoTopicName>/camera/depth/camera_info</depthImageInfoTopicName>
+        <pointCloudTopicName>/camera/depth_registered/points</pointCloudTopicName>
+        <frameName>camera_link_optical</frameName>
+        <pointCloudCutoff>0.12</pointCloudCutoff>
+        <pointCloudCutoffMax>3.0</pointCloudCutoffMax>
+        <distortionK1>0.00000001</distortionK1>
+        <distortionK2>0.00000001</distortionK2>
+        <distortionK3>0.00000001</distortionK3>
+        <distortionT1>0.00000001</distortionT1>
+        <distortionT2>0.00000001</distortionT2>
+        <CxPrime>0</CxPrime>
+        <Cx>0</Cx>
+        <Cy>0</Cy>
+        <focalLength>0</focalLength>
+        <hackBaseline>0</hackBaseline>
+      </plugin>
+    </sensor>
+  </gazebo>
+  <!-- USB Camera -->
+  <!-- !Here we rename camera1 to camera2 in order for the depth camera and usb camera to co-exist -->
   <gazebo reference="camera_link">
-    <sensor type="camera" name="camera1">
+    <!-- <sensor type="camera" name="camera1"> -->
+    <sensor type="camera" name="camera2">
       <update_rate>30.0</update_rate>
       <camera name="head">
@@ -93,11 +150,13 @@
         </noise>
       </camera>
-      <plugin name="camera_controller" filename="libgazebo_ros_camera.so">
+      <!-- <plugin name="camera_controller" filename="libgazebo_ros_camera.so"> -->
+      <plugin name="camera2_controller" filename="libgazebo_ros_camera.so">
         <alwaysOn>true</alwaysOn>
         <updateRate>0.0</updateRate>
-        <cameraName>camera1</cameraName>
+        <!-- <cameraName>camera1</cameraName> -->
+         <cameraName>camera2</cameraName>
         <imageTopicName>image_raw</imageTopicName>
         <cameraInfoTopicName>camera_info</cameraInfoTopicName>
-        <frameName>camera_link</frameName>
+        <frameName>camera2_link</frameName>
         <hackBaseline>0.07</hackBaseline>
         <distortionK1>0.0</distortionK1>

File: robots/archie_mw/xacros/properties.xacro (robot description, xacro)
@@ -33,4 +33,5 @@
     <xacro:property name="electronics_box_height" value="${100*SCALE_mm_to_m}" />
     <xacro:property name="electronics_box_half_height" value="${electronics_box_height/2}" />
+    <xacro:property name="electronics_box_z_offset" value="${chassis_center_to_base_footprint_z_offset + chassis_half_height}" />
     <xacro:property name="electronics_box_weight" value="${15}" /> <!-- in kg-->
     <!-- MOTOR WITH SUPPORT AND ELASTIC CLUTCH COUPLER DIMENSIONS  -->
@@ -55,5 +56,6 @@
     <xacro:property name="shaft_z_offset" value="${72.6*SCALE_mm_to_m}" /> <!--- From the ground to the middle of the shaft-->
     <!-- MECANUM WHEELS -->
-    <xacro:property name="wheel_diameter" value="${6*SCALE_in_to_m}" />
+    <!-- <xacro:property name="wheel_diameter" value="${6*SCALE_in_to_m}" /> -->
+    <xacro:property name="wheel_diameter" value="${152.4*SCALE_mm_to_m}" />
     <xacro:property name="wheel_radius" value="${wheel_diameter/2}" />
     <xacro:property name="wheel_width" value="${46*SCALE_mm_to_m}" />
@@ -63,4 +65,11 @@
     <!-- <xacro:property name="left_front_wheel_z_offset" value="${34.5*SCALE_mm_to_m}" /> -->
     <xacro:property name="left_front_wheel_z_offset" value="${72.6*SCALE_mm_to_m}" /> <!--- From the ground to the middle of the wheel-->
+    <!-- SENSORS -->
+    <xacro:property name="rplidar_a2_laser_beam_joint_x_offset" value="${0}" />
+    <xacro:property name="rplidar_a2_laser_beam_joint_y_offset" value="${0}" />
+    <xacro:property name="rplidar_a2_laser_beam_joint_z_offset" value="${electronics_box_z_offset+electronics_box_half_height+41*SCALE_mm_to_m}" /> <!--  From the electronics box middle point /> -->
+    <xacro:property name="rplidar_a2_mesh_X_offset" value="${*SCALE_mm_to_m}" />
+    <xacro:property name="rplidar_a2_mesh_Y_offset" value="${*SCALE_mm_to_m}" />
+    <xacro:property name="rplidar_a2_mesh_Z_offset" value="${*SCALE_mm_to_m}" />
     <!-- EUROPEAN STANDARD 2020 ALUMINIUM EXTRUSION PROFILE DIMENSIONS  -->
     <xacro:property name="profile_2020_width" value="${20*SCALE_mm_to_m}" />

Commit message: Add RPLidar A2 and replace bad tag in Gazebo world

File: robots/archie_mw/archie_mw.urdf.xacro (robot description, xacro)
@@ -19,4 +19,6 @@
   <!-- SENSORS -->
   <!-- <xacro:include filename="$(find archie_simulation)/robots/archie_mw/xacros/sick_S300.xacro" /> -->
+  <!-- rplidar_a2 gazebo reference -->
+  <xacro:include filename="$(find archie_simulation)/robots/archie_mw/xacros/rplidar_a2.gazebo.xacro" />
   <!-- Microscan - Comment/Uncomment if required -->
   <xacro:include filename="$(find archie_simulation)/robots/archie_mw/xacros/micro_scan.xacro" />
@@ -92,10 +94,10 @@
 <!-- ####################### -->
   <!-- Sensors -->
-  <xacro:fixed_joint name="rplidar_a2_laser_beam_joint" parent_name="electronics_box" child_name="rplidar_a2_laser_beam_link" color="Red">
+  <!-- <xacro:fixed_joint name="rplidar_a2_laser_beam_joint" parent_name="electronics_box" child_name="rplidar_a2_laser_beam_link" color="Red">
     <origin xyz="${rplidar_a2_laser_beam_joint_x_offset} ${rplidar_a2_laser_beam_joint_y_offset} ${electronics_box_height}" rpy="0 0 ${ROTATE_180_DEGREES}" />
   </xacro:fixed_joint>
-  <xacro:box_link name="rplidar_a2_laser_beam_link" lenght="${0.041}" width="${0.041}" height="${0.001}" mass="${0.005}" color="Red">
+  <xacro:box_link name="rplidar_a2_laser_beam_link" lenght="${0.041}" width="${0.041}" height="${0.001}" mass="${0.005}" color="Blue">
     <origin xyz="0 0 0" rpy="0 0 0" />
-  </xacro:box_link>
+  </xacro:box_link> -->
   <!-- <xacro:fixed_joint name="rplidar_a2_laser_beam_fom_base_link_joint" parent_name="base_link" child_name="rplidar_a2_laser_beam_fom_base_link_link" color="Red">
     <origin xyz="${rplidar_a2_laser_beam_joint_x_offset} ${rplidar_a2_laser_beam_joint_y_offset} ${230.7*SCALE_mm_to_m}" rpy="0 0 ${ROTATE_180_DEGREES}" />
@@ -104,10 +106,38 @@
     <origin xyz="0 0 0" rpy="0 0 0" />
   </xacro:box_link> -->
-  <xacro:sick_laser_v0 name="lidar_1" parent="base_link" ros_topic="lidar_1/scan_filtered">
+<joint name="rplidar_joint" type="fixed"> <!-- Seting the joint at the laser beam plane -->
+    <axis xyz="0 1 0" />
+    <!-- <origin xyz="0.02 0 0.058" rpy="0 0 3.14"/> -->
+    <origin xyz="${rplidar_a2_laser_beam_joint_x_offset} ${rplidar_a2_laser_beam_joint_y_offset} ${electronics_box_height+0.0308}" rpy="0 0 ${ROTATE_180_DEGREES}" />
+    <parent link="electronics_box"/>
+    <child link="laser"/>
+  </joint>
+  <!-- rplidar Laser -->
+  <link name="laser">
+    <collision>
+      <origin xyz="0 0 -0.0308" rpy="1.5707 0 4.71"/> <!-- Move the mesh down on Z axis, as the joint is at the laser beam plane -->
+      <geometry>
+        <mesh filename="package://archie_simulation/robots/archie_mw/meshes/rplidar.dae" scale="0.001 0.001 0.001" />
+      </geometry>
+    </collision>
+    <visual>
+      <origin xyz="0 0 -0.0308" rpy="1.5707 0 4.71"/>
+      <geometry>
+        <mesh filename="package://archie_simulation/robots/archie_mw/meshes/rplidar.dae" scale="0.001 0.001 0.001" />
+      </geometry>
+    </visual>
+    <inertial>
+      <mass value="1e-5" />
+      <origin xyz="0 0 -0.0308" rpy="1.5707 0 4.71"/>
+      <inertia ixx="0" ixy="0" ixz="0" iyy="0" iyz="0" izz="0" />
+    </inertial>
+  </link>
+<!-- COMMENT THE FORMER SICK LIDARS -->
+  <!-- <xacro:sick_laser_v0 name="lidar_1" parent="base_link" ros_topic="lidar_1/scan_filtered">
     <origin xyz="0.442 0 0.372" rpy="0 0 0" />
   </xacro:sick_laser_v0>
   <xacro:sick_laser_v0 name="lidar_2" parent="base_link" ros_topic="lidar_2/scan_filtered">
     <origin xyz="-0.442 0 0.372" rpy="0 0 3.14" />
-  </xacro:sick_laser_v0>
+  </xacro:sick_laser_v0> -->
   <!--+++++++++++++++++++ IMU ++++++++++++++++++++++++-->
   <!-- Comment or uncomment based on your requirement -->
