Commit message: Add wheel meshes and torso standoff (pole). Position RPLidar at the front

File: robots/archie_mw/archie_mw.urdf.xacro (robot description, xacro)
@@ -67,4 +67,51 @@
     <origin xyz="0 0 0" rpy="0 0 0" />
   </xacro:box_link>
+<!-- **** ROBOT TORSO STANDOFF (POLE) height = 406.8 mm ****  -->
+<!-- The heap is located at about 0.53 of the human body lenght -->
+<!-- Robot haight - 1200 mm, Heap height from the ground = 1200 mm * 0.53 = 636 mm -->
+<!-- Torso standoff height is 636 mm - base_plate_botom_from_base_frame_Z_offset - chassis_height - electronics_box_height  -->
+<!-- standoff_height = 636 - 40.2 - 89 - 100 = 406.8 -->
+<!-- aluminium profile 40x40 will be used weight of the profile is: 2.45 kg/meter -->
+<!-- ! The Joint is positioned on top plane of the electronics box module -->
+  <xacro:fixed_joint name="torso_standoff" parent_name="electronics_box" child_name="torso_standoff" color="Grey">
+    <origin xyz="0 0 ${100*SCALE_mm_to_m}" rpy="0 0 0" />
+  </xacro:fixed_joint>
+<!-- ! Mass of the aluminium profile is 2.45kg per meter -->
+  <xacro:box_link name="torso_standoff" lenght="${40*SCALE_mm_to_m}" width="${40*SCALE_mm_to_m}" height="${406.8*SCALE_mm_to_m}" mass="${2.45*0.4068}" color="Grey">
+    <origin xyz="0 0 ${406.8*SCALE_mm_to_m/2}" rpy="0 0 0" />
+  </xacro:box_link>
+<!-- WHEEL SHAFTS -->
+<!-- Invoke shaft_joint macros for the front left shaft -->
+    <xacro:shaft_joint name="front_left">
+      <origin xyz="${shaft_x_offset} ${shaft_y_offset} ${shaft_z_offset}" rpy="0 0 0" />
+    </xacro:shaft_joint>
+<!-- Invoke shaft_link macros for the front left shaft -->
+    <xacro:shaft_link name="front_left" radius="${shaft_radius}" lenght="${shaft_lenght}" mass="${shaft_mass}" color="Black">
+      <origin xyz="0 ${shaft_half_lenght} 0" rpy="${ROTATE_90_DEGREES} 0 0" />
+    </xacro:shaft_link>
+<!-- Invoke shaft_joint macros for the back left shaft -->
+    <xacro:shaft_joint name="back_left">
+      <origin xyz="${-shaft_x_offset} ${shaft_y_offset} ${shaft_z_offset}" rpy="0 0 0" />
+    </xacro:shaft_joint>
+<!-- Invoke shaft_link macros for the back left shaft -->
+    <xacro:shaft_link name="back_left" radius="${shaft_radius}" lenght="${shaft_lenght}" mass="${shaft_mass}" color="Black">
+      <origin xyz="0 ${shaft_half_lenght} 0" rpy="${ROTATE_90_DEGREES} 0 0" />
+    </xacro:shaft_link>
+<!-- Invoke shaft_joint macros for the front right shaft -->
+    <xacro:shaft_joint name="front_right">
+      <origin xyz="${shaft_x_offset} ${-shaft_y_offset} ${shaft_z_offset}" rpy="0 0 0" />
+    </xacro:shaft_joint>
+<!-- Invoke shaft_link macros for the front right shaft -->
+    <xacro:shaft_link name="front_right" radius="${shaft_radius}" lenght="${shaft_lenght}" mass="${shaft_mass}" color="Black">
+      <origin xyz="0 ${-shaft_half_lenght} 0" rpy="${ROTATE_90_DEGREES} 0 0" />
+    </xacro:shaft_link>
+<!-- Invoke shaft_joint macros for the back right shaft -->
+    <xacro:shaft_joint name="back_right">
+      <origin xyz="${-shaft_x_offset} ${-shaft_y_offset} ${shaft_z_offset}" rpy="0 0 0" />
+    </xacro:shaft_joint>
+<!-- Invoke shaft_link macros for the back right shaft -->
+    <xacro:shaft_link name="back_right" radius="${shaft_radius}" lenght="${shaft_lenght}" mass="${shaft_mass}" color="Black">
+      <origin xyz="0 ${-shaft_half_lenght} 0" rpy="${ROTATE_90_DEGREES} 0 0" />
+    </xacro:shaft_link>
   <!-- Invoke Wheel Macros -->
   <xacro:mecanum_wheel_152 name="archie_mw_mecanum_wheel_front_left" parent="base_footprint" diameter="${wheel_diameter}" width="${wheel_width}" mass="${wheel_weight}" color="White"
@@ -73,15 +120,15 @@
     <origin xyz="${left_front_wheel_x_offset} ${left_front_wheel_y_offset+shaft_lenght} ${left_front_wheel_z_offset}" rpy="0 0 0" />
   </xacro:mecanum_wheel_152>
-  <xacro:mecanum_wheel_152 name="archie_mw_mecanum_wheel_front_right" parent="base_link" diameter="${wheel_diameter}" width="${wheel_width}" mass="${wheel_weight}" color="White"
+  <xacro:mecanum_wheel_152 name="archie_mw_mecanum_wheel_front_right" parent="base_footprint" diameter="${wheel_diameter}" width="${wheel_width}" mass="${wheel_weight}" color="White"
       mesh_file_name="package://archie_simulation/robots/archie_mw/meshes/mecanum_wheel_right.STL" mesh_scale_x="${1*SCALE_mm_to_m}"
       mesh_scale_y="${0.92*SCALE_mm_to_m}" mesh_scale_z="${1.52*SCALE_mm_to_m}">
     <origin xyz="${left_front_wheel_x_offset} ${-(left_front_wheel_y_offset+shaft_lenght)} ${left_front_wheel_z_offset}" rpy="0 0 0" />
   </xacro:mecanum_wheel_152>
-  <xacro:mecanum_wheel_152 name="archie_mw_mecanum_wheel_back_left" parent="base_link" diameter="${wheel_diameter}" width="${wheel_width}" mass="${wheel_weight}" color="White"
+  <xacro:mecanum_wheel_152 name="archie_mw_mecanum_wheel_back_left" parent="base_footprint" diameter="${wheel_diameter}" width="${wheel_width}" mass="${wheel_weight}" color="White"
       mesh_file_name="package://archie_simulation/robots/archie_mw/meshes/mecanum_wheel_left.STL" mesh_scale_x="${1*SCALE_mm_to_m}"
       mesh_scale_y="${0.92*SCALE_mm_to_m}" mesh_scale_z="${1.52*SCALE_mm_to_m}">
     <origin xyz="${-left_front_wheel_x_offset} ${left_front_wheel_y_offset+shaft_lenght} ${left_front_wheel_z_offset}" rpy="0 0 0" />
   </xacro:mecanum_wheel_152>
-  <xacro:mecanum_wheel_152 name="archie_mw_mecanum_wheel_back_right" parent="base_link" diameter="${wheel_diameter}" width="${wheel_width}" mass="${wheel_weight}" color="White"
+  <xacro:mecanum_wheel_152 name="archie_mw_mecanum_wheel_back_right" parent="base_footprint" diameter="${wheel_diameter}" width="${wheel_width}" mass="${wheel_weight}" color="White"
       mesh_file_name="package://archie_simulation/robots/archie_mw/meshes/mecanum_wheel_right.STL" mesh_scale_x="${1*SCALE_mm_to_m}"
       mesh_scale_y="${0.92*SCALE_mm_to_m}" mesh_scale_z="${1.52*SCALE_mm_to_m}">
@@ -106,8 +153,10 @@
     <origin xyz="0 0 0" rpy="0 0 0" />
   </xacro:box_link> -->
+<!--  **** RP LIDAR A2 **** -->
+<!-- ! The Joint is positioned at the laser beam plane, which is offset 30.8 mm from the electronics box top-->
 <joint name="rplidar_joint" type="fixed"> <!-- Seting the joint at the laser beam plane -->
     <axis xyz="0 1 0" />
     <!-- <origin xyz="0.02 0 0.058" rpy="0 0 3.14"/> -->
-    <origin xyz="${rplidar_a2_laser_beam_joint_x_offset} ${rplidar_a2_laser_beam_joint_y_offset} ${electronics_box_height+0.0308}" rpy="0 0 ${ROTATE_180_DEGREES}" />
+    <origin xyz="${rplidar_a2_laser_beam_joint_x_offset} ${rplidar_a2_laser_beam_joint_y_offset} ${rplidar_a2_laser_beam_joint_z_offset}" rpy="${rplidar_a2_laser_beam_joint_roll} ${rplidar_a2_laser_beam_joint_pitch} ${rplidar_a2_laser_beam_joint_yaw}" />
     <parent link="electronics_box"/>
     <child link="laser"/>

File: robots/archie_mw/xacros/archie_mw_gazebo.xacro (robot description, xacro)
@@ -2,9 +2,45 @@
 <robot name="archie_mw" xmlns:xacro="http://www.ros.org/wiki/xacro">
 <!-- TODO Is this gravity and self colide needed????????????????/ -->
-   <gazebo reference="base_link">
+  <gazebo reference="base_link">
     <gravity>true</gravity>
     <self_collide>false</self_collide>
   </gazebo>
+<!-- CHASSIS  -->
+  <gazebo reference="base_footprint">
+    <material>Gazebo/Grey</material>
+  </gazebo>
+<!-- ELECTRONICS BOX  -->
+  <gazebo reference="electronics_box">
+    <material>Gazebo/DarkGrey</material>
+  </gazebo>
+<!-- WHEEL SHAFTS  -->
+  <gazebo reference="front_left_wheel_shaft_link">
+    <material>Gazebo/Black</material>
+  </gazebo>
+  <gazebo reference="back_left_wheel_shaft_link">
+    <material>Gazebo/Black</material>
+  </gazebo>
+  <gazebo reference="front_right_wheel_shaft_link">
+    <material>Gazebo/Black</material>
+  </gazebo>
+  <gazebo reference="back_right_wheel_shaft_link">
+    <material>Gazebo/Black</material>
+  </gazebo>
+<!-- WHEELS  -->
+  <gazebo reference="archie_mw_mecanum_wheel_front_left_link">
+    <material>Gazebo/Grey</material>
+  </gazebo>
+  <gazebo reference="archie_mw_mecanum_wheel_back_left_link">
+    <material>Gazebo/Grey</material>
+  </gazebo>
+  <gazebo reference="archie_mw_mecanum_wheel_front_right_link">
+    <material>Gazebo/Grey</material>
+  </gazebo>
+  <gazebo reference="archie_mw_mecanum_wheel_back_right_link">
+    <material>Gazebo/Grey</material>
+  </gazebo>
   <!-- Lidar sensors -->
+<!-- RPlIDAR a2 VISUAL is rplidar_a2.gazebo.xacro -->
+<!-- SICK-3000  -->
   <gazebo reference="lidar_1_link">
       <sensor type="ray" name="lidar_1_sensor">

File: robots/archie_mw/xacros/mecanum_wheel.xacro (robot description, xacro)
@@ -1,4 +1,33 @@
 <?xml version="1.0"?>
 <robot xmlns:xacro="http://www.ros.org/wiki/xacro" name="archie_mw">
+  <xacro:macro name="shaft_joint" params="name *origin">
+  <joint name="${name}_wheel_shaft_joint" type="fixed">
+    <!-- <parent link="base_link"/> -->
+    <parent link="base_footprint"/>
+    <child link="${name}_wheel_shaft_link" />
+    <xacro:insert_block name="origin" />
+  </joint>
+  </xacro:macro>
+  <xacro:macro name="shaft_link" params="name radius lenght mass color *origin">
+  <link name="${name}_wheel_shaft_link">
+    <visual>
+      <xacro:insert_block name="origin" />
+      <geometry>
+        <cylinder radius="${radius}" length="${lenght}"/>
+      </geometry>
+      <material name="${color}" />
+    </visual>
+    <collision>
+      <xacro:insert_block name="origin" />
+      <geometry>
+        <cylinder radius="${radius}" length="${lenght}"/>
+      </geometry>
+    </collision>
+    <xacro:cylinder_inertial_with_origin radius="${radius}" length="${lenght}" mass="${mass}">
+      <xacro:insert_block name="origin" />
+    </xacro:cylinder_inertial_with_origin>
+  </link>
+  </xacro:macro>
+<!-- ################### -->
   <xacro:macro name="mecanum_wheel_152" params="name parent *origin mass color diameter width mesh_file_name mesh_scale_x mesh_scale_y mesh_scale_z">
    <joint name="${name}_joint" type="revolute">
@@ -23,5 +52,6 @@
     </xacro:cylinder_inertial_with_origin>
     <visual>
-     <origin xyz="0 0 0" rpy="${ROTATE_90_DEGREES} 0 0"/>
+     <!-- <origin xyz="0 0 0" rpy="${ROTATE_90_DEGREES} 0 0"/> -->
+     <origin xyz="0 0 0" rpy="0 0 0"/>
     <!-- <xacro:insert_block name="visual_origin" />      -->
     <!-- <origin xyz="0 0 0" rpy="0 0 0"/> -->
@@ -29,6 +59,6 @@
         <!-- <mesh filename="package://archie_simulation/robots/mpo_500/meshes/MPO-500-WHEEL.dae" scale="0.001 0.001 0.001"/> -->
         <!-- <mesh filename="package://archie_simulation/robots/archie_mw/meshes/mecanum_wheel_left.STL" scale="0.001 0.001 0.001"/> -->
-        <!-- <mesh filename="${mesh_file_name}" scale="${mesh_scale_x} ${mesh_scale_y} ${mesh_scale_z}"/> -->
-      <cylinder radius="0.076" length="0.046"/>
+        <mesh filename="${mesh_file_name}" scale="${mesh_scale_x} ${mesh_scale_y} ${mesh_scale_z}"/>
+      <!-- <cylinder radius="0.076" length="0.046"/> -->
       <!-- <cylinder radius="${diameter/2}" length="${width}"/> -->
     </geometry>

File: robots/archie_mw/xacros/properties.xacro (robot description, xacro)
@@ -66,10 +66,18 @@
     <xacro:property name="left_front_wheel_z_offset" value="${72.6*SCALE_mm_to_m}" /> <!--- From the ground to the middle of the wheel-->
     <!-- SENSORS -->
-    <xacro:property name="rplidar_a2_laser_beam_joint_x_offset" value="${0}" />
+    <!--  **** RP LIDAR A2 **** -->
+    <!-- ! The Joint is positioned at the laser beam plane, which is offset 30.8 mm from the electronics box top-->
+    <!-- Position the RP Lidar 10 mm from the front edge of the electronics box, to avoid the chance of collision, just in case. -->
+    <!-- RP Lidar's /diameter 75.7 mm/ center point needs to be at x = (337.5 - 10) - (75.7/2) = 289.65 mm from the box center -->
+    <xacro:property name="rplidar_a2_laser_beam_joint_x_offset" value="${289.65*SCALE_mm_to_m}" />
     <xacro:property name="rplidar_a2_laser_beam_joint_y_offset" value="${0}" />
-    <xacro:property name="rplidar_a2_laser_beam_joint_z_offset" value="${electronics_box_z_offset+electronics_box_half_height+41*SCALE_mm_to_m}" /> <!--  From the electronics box middle point /> -->
-    <xacro:property name="rplidar_a2_mesh_X_offset" value="${*SCALE_mm_to_m}" />
-    <xacro:property name="rplidar_a2_mesh_Y_offset" value="${*SCALE_mm_to_m}" />
-    <xacro:property name="rplidar_a2_mesh_Z_offset" value="${*SCALE_mm_to_m}" />
+    <!-- The Z offset is positioning the joint at the laser beam plane -->
+    <xacro:property name="rplidar_a2_laser_beam_joint_z_offset" value="${electronics_box_height+0.0308}" />
+    <xacro:property name="rplidar_a2_laser_beam_joint_roll" value="${0}" />
+    <xacro:property name="rplidar_a2_laser_beam_joint_pitch" value="${0}" />
+    <xacro:property name="rplidar_a2_laser_beam_joint_yaw" value="${ROTATE_180_DEGREES}" />
+    <xacro:property name="rplidar_a2_mesh_X_offset" value="${0*SCALE_mm_to_m}" />
+    <xacro:property name="rplidar_a2_mesh_Y_offset" value="${0*SCALE_mm_to_m}" />
+    <xacro:property name="rplidar_a2_mesh_Z_offset" value="${0*SCALE_mm_to_m}" />
     <!-- EUROPEAN STANDARD 2020 ALUMINIUM EXTRUSION PROFILE DIMENSIONS  -->
     <xacro:property name="profile_2020_width" value="${20*SCALE_mm_to_m}" />

File: robots/archie_mw/xacros/rplidar_a2.gazebo.xacro (robot description, xacro)
@@ -106,4 +106,5 @@
       </plugin>
     </sensor>
+    <material>Gazebo/Grey</material>
   </gazebo>
   <!-- RpLidar A3 using CPU -->

Commit message: Add side boxes to mimic the mobile base shape shape

File: robots/archie_mw/archie_mw.urdf.xacro (robot description, xacro)
@@ -67,4 +67,33 @@
     <origin xyz="0 0 0" rpy="0 0 0" />
   </xacro:box_link>
+  <!-- **** SIDE BOXES (COVERS) ****  -->
+  <!-- Lower part of the side box -->
+  <xacro:fixed_joint name="left_lower_side_box_joint" parent_name="base_link" child_name="left_lower_side_box" color="Grey">
+    <origin xyz="0 ${electronics_box_width/2+34.5*SCALE_mm_to_m} ${(97.05-41.7-14)*SCALE_mm_to_m}" rpy="0 0 0" />
+  </xacro:fixed_joint>
+  <xacro:box_link name="left_lower_side_box" lenght="${480*SCALE_mm_to_m}" width="${69*SCALE_mm_to_m}" height="${110.7*SCALE_mm_to_m}" mass="${2}" color="Yellow">
+    <origin xyz="0 0 0" rpy="0 0 0" />
+  </xacro:box_link>
+  <!-- Top part of the side box -->
+  <xacro:fixed_joint name="left_top_side_box_joint" parent_name="base_link" child_name="left_top_side_box" color="Grey">
+    <origin xyz="0 ${electronics_box_width/2+34.5*SCALE_mm_to_m} ${(110.7+40.2)*SCALE_mm_to_m}" rpy="0 0 0" />
+  </xacro:fixed_joint>
+  <xacro:box_link name="left_top_side_box" lenght="${electronics_box_lenght}" width="${69*SCALE_mm_to_m}" height="${80*SCALE_mm_to_m}" mass="${2}" color="Yellow">
+    <origin xyz="0 0 0" rpy="0 0 0" />
+  </xacro:box_link>
+  <!-- Lower part of the right side box -->
+  <xacro:fixed_joint name="right_lower_side_box_joint" parent_name="base_link" child_name="right_lower_side_box" color="Grey">
+    <origin xyz="0 ${-(electronics_box_width/2+34.5*SCALE_mm_to_m)} ${(97.05-41.7-14)*SCALE_mm_to_m}" rpy="0 0 0" />
+  </xacro:fixed_joint>
+  <xacro:box_link name="right_lower_side_box" lenght="${480*SCALE_mm_to_m}" width="${69*SCALE_mm_to_m}" height="${110.7*SCALE_mm_to_m}" mass="${2}" color="Yellow">
+    <origin xyz="0 0 0" rpy="0 0 0" />
+  </xacro:box_link>
+  <!-- Top part of the right side box -->
+  <xacro:fixed_joint name="right_top_side_box_joint" parent_name="base_link" child_name="right_top_side_box" color="Grey">
+    <origin xyz="0 ${-(electronics_box_width/2+34.5*SCALE_mm_to_m)} ${(110.7+40.2)*SCALE_mm_to_m}" rpy="0 0 0" />
+  </xacro:fixed_joint>
+  <xacro:box_link name="right_top_side_box" lenght="${electronics_box_lenght}" width="${69*SCALE_mm_to_m}" height="${80*SCALE_mm_to_m}" mass="${2}" color="Yellow">
+    <origin xyz="0 0 0" rpy="0 0 0" />
+  </xacro:box_link>
 <!-- **** ROBOT TORSO STANDOFF (POLE) height = 406.8 mm ****  -->
 <!-- The heap is located at about 0.53 of the human body lenght -->

File: robots/archie_mw/xacros/archie_mw_gazebo.xacro (robot description, xacro)
@@ -12,5 +12,18 @@
 <!-- ELECTRONICS BOX  -->
   <gazebo reference="electronics_box">
+    <material>Gazebo/Yellow</material>
+  </gazebo>
+<!-- EXTENSION SIDE BOXES  -->
+  <gazebo reference="left_lower_side_box">
     <material>Gazebo/DarkGrey</material>
+  </gazebo>
+  <gazebo reference="left_top_side_box">
+    <material>Gazebo/Yellow</material>
+  </gazebo>
+  <gazebo reference="right_lower_side_box">
+    <material>Gazebo/DarkGrey</material>
+  </gazebo>
+  <gazebo reference="right_top_side_box">
+    <material>Gazebo/Yellow</material>
   </gazebo>
 <!-- WHEEL SHAFTS  -->
@@ -162,4 +175,5 @@
       </plugin>
     </sensor>
+    <material>Gazebo/Yellow</material>
   </gazebo>
   <!-- USB Camera -->

File: robots/archie_mw/xacros/depth_camera.xacro (robot description, xacro)
@@ -31,5 +31,5 @@
 			      	<mesh filename="package://archie_simulation/robots/archie_mw/meshes/realsense_d435.dae"/>
 			      </geometry>
-			      <material name="red">
+			      <material name="Red">
 			      	<color rgba="1 0 0 1" />
 			      </material>

Commit message: Add table docking world

File: robots/archie_mw/archie_mw.urdf.xacro (robot description, xacro)
@@ -105,11 +105,11 @@
 <!-- aluminium profile 40x40 will be used weight of the profile is: 2.45 kg/meter -->
 <!-- ! The Joint is positioned on top plane of the electronics box module -->
-  <xacro:fixed_joint name="torso_standoff" parent_name="electronics_box" child_name="torso_standoff" color="Grey">
+  <!-- <xacro:fixed_joint name="torso_standoff" parent_name="electronics_box" child_name="torso_standoff" color="Grey">
     <origin xyz="0 0 ${100*SCALE_mm_to_m}" rpy="0 0 0" />
-  </xacro:fixed_joint>
+  </xacro:fixed_joint> -->
 <!-- ! Mass of the aluminium profile is 2.45kg per meter -->
-  <xacro:box_link name="torso_standoff" lenght="${40*SCALE_mm_to_m}" width="${40*SCALE_mm_to_m}" height="${406.8*SCALE_mm_to_m}" mass="${2.45*0.4068}" color="Grey">
+  <!-- <xacro:box_link name="torso_standoff" lenght="${40*SCALE_mm_to_m}" width="${40*SCALE_mm_to_m}" height="${406.8*SCALE_mm_to_m}" mass="${2.45*0.4068}" color="Grey">
     <origin xyz="0 0 ${406.8*SCALE_mm_to_m/2}" rpy="0 0 0" />
-  </xacro:box_link>
+  </xacro:box_link> -->
 <!-- ORBBEC ASTRA RGBD CAMERA (ONLY VISUAL) -->
   <xacro:astra_depth_camera name="astra_camera" >

File: robots/archie_mw/xacros/astra_rgbd_macro.xacro (robot description, xacro)
@@ -22,4 +22,6 @@
       <geometry>
         <mesh filename="package://archie_simulation/robots/archie_mw/meshes/astra.dae" scale="0.001 0.001 0.001" />
+		<!-- <mesh filename="package://archie_simulation/robots/archie_mw/meshes/realsense_d435.dae"/> -->
+		<!-- <mesh filename="package://archie_simulation/robots/archie_mw/meshes/IntelRealsense_D435_Multibody.stl" scale="0.001 0.001 0.001"/> -->
       </geometry>
     </visual>
@@ -30,5 +32,5 @@
     </inertial>
   </link>
-  <joint name="astra_camera_optical_joint" type="fixed">
+  <!-- <joint name="astra_camera_optical_joint" type="fixed">
     <origin xyz="0 0 0" rpy="${-pi/2} 0 ${-pi/2}"/>
     <parent link="astra_camera_link"/>
@@ -42,6 +44,6 @@
     <child link="astra_camera_depth_frame"/>
   </joint>
-  <link name="astra_acamera_depth_frame">
-  </link>
+  <link name="astra_camera_depth_frame">
+  </link> -->
     </xacro:macro>
 </robot>
