Commit message: Change transmission name and data in other packages, BUG model flying?

File: robots/archie_mw/archie_mw.urdf copy.xacro (robot description, xacro)
@@ -50,9 +50,8 @@
   </gazebo> -->
   <link name="base_link" />
-    <!-- color="Yellow" z_offset="${chassis_center_to_base_footprint_z_offset}"> -->
   <!-- Base link macro -->
   <xacro:archie_mw_base name="base_footprint" parent="base_link" lenght="${chassis_lenght}"
     width="${chassis_width}" height="${chassis_height}" mass="${chassis_weight}"
-    color="Yellow" z_offset="${chassis_bottom_z_offset}">
+    color="Yellow" z_offset="${chassis_center_to_base_footprint_z_offset}">
     <joint_origin xyz="0 0 0" rpy="0 0 0" />
   </xacro:archie_mw_base>

File: robots/archie_mw/xacros/archie_mw_colors_gazebo.xacro (robot description, xacro)
@@ -1,27 +1,3 @@
 <?xml version="1.0"?>
 <robot name="archie_mw" xmlns:xacro="http://www.ros.org/wiki/xacro">
-  <!-- All static links get collapsed down to base_link in Gazebo, so that's
-       the one to apply the colour to (in Gazebo 5+). -->
- <!-- !NOTE base_link acts as base_frame in this project!!! Reverse them later!!! -->
-  <!-- <gazebo reference="base_link">
-    <material>Gazebo/Yellow</material>
-    <gravity>true</gravity>
-  </gazebo> -->
-    <gazebo reference="base_link">
-        <gravity>true</gravity>
-        <self_collide>false</self_collide>
-        <material>Gazebo/Yellow</material>
-    </gazebo>
- <!-- !NOTE base_footprint represents the chassis this project!!! -->
-    <gazebo reference="base_footprint">
-        <material>Gazebo/DarkGrey</material>
-        <gravity>true</gravity>
-    </gazebo>
-  <!-- <gazebo reference="base_footprint">
-    <material>Gazebo/DarkGrey</material>
-  </gazebo> -->
-  <!-- <gazebo reference="electronics_module_link">
-    <material>Gazebo/Grey</material>
-  </gazebo> -->
-<!-- ######### WHEELS - Gazebo  mu1, mu2 and material are defined in mecanum_wheel.xacro -->
 </robot>

File: robots/archie_mw/xacros/archie_mw_gazebo.xacro (robot description, xacro)
@@ -1,12 +1,24 @@
 <?xml version="1.0"?>
 <robot name="archie_mw" xmlns:xacro="http://www.ros.org/wiki/xacro">
+  <!-- All static links get collapsed down to base_link in Gazebo, so that's
+       the one to apply the colour to (in Gazebo 5+). -->
+ <!-- !NOTE base_link acts as base_frame in this project!!! Reverse them later!!! -->
+  <gazebo reference="base_link">
+    <material>Gazebo/Yellow</material>
+    <gravity>true</gravity>
+  </gazebo>
 <!-- TODO Is this gravity and self colide needed????????????????/ -->
-  <gazebo reference="base_link">
-    <gravity>true</gravity>
-    <self_collide>false</self_collide>
-  </gazebo>
+    <!-- <gazebo reference="base_link">
+        <gravity>true</gravity>
+        <self_collide>false</self_collide>
+    </gazebo> -->
+ <!-- !NOTE base_footprint represents the chassis this project!!! -->
 <!-- CHASSIS  -->
+    <!-- <gazebo reference="base_footprint">
+        <material>Gazebo/DarkGrey</material>
+        <gravity>true</gravity>
+    </gazebo> -->
   <gazebo reference="base_footprint">
-    <material>Gazebo/Grey</material>
+    <material>Gazebo/DarkGrey</material>
   </gazebo>
 <!-- ELECTRONICS BOX  -->
@@ -41,5 +53,7 @@
   </gazebo>
 <!-- WHEELS  -->
-  <gazebo reference="archie_mw_mecanum_wheel_front_left_link">
+<!-- !######### WHEELS - Gazebo  mu1, mu2 and material are defined in
+     ! mecanum_wheel.xacro -->
+  <!-- <gazebo reference="archie_mw_mecanum_wheel_front_left_link">
     <material>Gazebo/Grey</material>
   </gazebo>
@@ -52,5 +66,5 @@
   <gazebo reference="archie_mw_mecanum_wheel_back_right_link">
     <material>Gazebo/Grey</material>
-  </gazebo>
+  </gazebo> -->
   <!-- Lidar sensors -->
 <!-- RPlIDAR a2 VISUAL is rplidar_a2.gazebo.xacro -->
@@ -184,5 +198,7 @@
       <update_rate>30.0</update_rate>
       <camera name="head">
-        <horizontal_fov>1.3962634</horizontal_fov>
+        <!-- <horizontal_fov>1.3962634</horizontal_fov> -->
+        <!-- !Copied from the depth camera values??? -->
+      <hfov>70</hfov>
         <image>
           <width>800</width>
