Commit message: Cahnge RPLidar topic and frame. Change map arg in amcl.launch

File: robots/archie_mw/xacros/rplidar_a2.gazebo.xacro (robot description, xacro)
@@ -7,4 +7,41 @@
     stddev of 0.01m will put 99.7% of samples within 0.03m of the true
     reading. -->
+  <!-- RpLidar A2 using CPU -->
+  <gazebo reference="laser">
+    <!-- <sensor type="ray" name="head_rplidar_sensor"> -->
+    <!-- Change the name to match the former SICK laser name -->
+    <sensor type="ray" name="lidar_1_sensor">
+      <pose>0 0 0.06 0 0 0</pose>
+      <visualize>false</visualize>
+      <update_rate>40</update_rate>
+      <ray>
+        <scan>
+          <horizontal>
+            <samples>720</samples>
+            <resolution>1</resolution>
+            <min_angle>-3.14159265</min_angle>
+            <max_angle>3.14159265</max_angle>
+          </horizontal>
+        </scan>
+        <range>
+          <min>0.2</min>
+          <max>12.0</max>
+          <resolution>0.01</resolution>
+        </range>
+        <noise>
+          <type>gaussian</type>
+          <mean>0.0</mean>
+          <stddev>0.01</stddev>
+        </noise>
+      </ray>
+      <plugin name="gazebo_ros_head_rplidar_controller" filename="libgazebo_ros_laser.so">
+        <!-- <topicName>scan</topicName> -->
+        <!-- Change the sacan topic to match the former SICK laser 1 -->
+        <topicName>lidar_1/scan_filtered</topicName>
+        <frameName>laser</frameName>
+      </plugin>
+    </sensor>
+    <material>Gazebo/Grey</material>
+  </gazebo>
   <!-- RpLidar A2 using GPU -->
   <!--<gazebo reference="laser">
@@ -71,41 +108,4 @@
     </sensor>
   </gazebo> -->
-  <!-- RpLidar A2 using CPU -->
-  <gazebo reference="laser">
-    <!-- <sensor type="ray" name="head_rplidar_sensor"> -->
-    <!-- Change the name to match the former SICK laser name -->
-    <sensor type="ray" name="lidar_1_sensor">
-      <pose>0 0 0.06 0 0 0</pose>
-      <visualize>false</visualize>
-      <update_rate>40</update_rate>
-      <ray>
-        <scan>
-          <horizontal>
-            <samples>720</samples>
-            <resolution>1</resolution>
-            <min_angle>-3.14159265</min_angle>
-            <max_angle>3.14159265</max_angle>
-          </horizontal>
-        </scan>
-        <range>
-          <min>0.2</min>
-          <max>12.0</max>
-          <resolution>0.01</resolution>
-        </range>
-        <noise>
-          <type>gaussian</type>
-          <mean>0.0</mean>
-          <stddev>0.01</stddev>
-        </noise>
-      </ray>
-      <plugin name="gazebo_ros_head_rplidar_controller" filename="libgazebo_ros_laser.so">
-        <!-- <topicName>scan</topicName> -->
-        <!-- Change the sacan topic to match the former SICK laser 1 -->
-        <topicName>lidar_1/scan_filtered</topicName>
-        <frameName>laser</frameName>
-      </plugin>
-    </sensor>
-    <material>Gazebo/Grey</material>
-  </gazebo>
   <!-- RpLidar A3 using CPU -->
   <!-- <gazebo reference="laser">
