Commit message: Correct typo arche_mb to archie_mb in all files

File: robots/archie_mb/archie_mb.urdf.xacro (robot description, xacro)
@@ -1,36 +1,36 @@
 <?xml version="1.0" ?>
-<robot name="arche_mb" xmlns:xacro="http://www.ros.org/wiki/xacro">
+<robot name="archie_mb" xmlns:xacro="http://www.ros.org/wiki/xacro">
   <!-- PROPERTIES -->
-  <xacro:include filename="$(find archie_simulation)/robots/arche_mb/xacros/properties.xacro" />
+  <xacro:include filename="$(find archie_simulation)/robots/archie_mb/xacros/properties.xacro" />
   <!-- MATERIALS -->
-  <xacro:include filename="$(find archie_simulation)/robots/arche_mb/xacros/materials.xacro" />
+  <xacro:include filename="$(find archie_simulation)/robots/archie_mb/xacros/materials.xacro" />
   <!-- INERTIAL CALCULATIONS -->
-  <xacro:include filename="$(find archie_simulation)/robots/arche_mb/xacros/inertial_calc_macros.xacro" />
+  <xacro:include filename="$(find archie_simulation)/robots/archie_mb/xacros/inertial_calc_macros.xacro" />
   <!--GAZEBO REFERENCES -->
-  <xacro:include filename="$(find archie_simulation)/robots/arche_mb/xacros/arche_mb_gazebo.xacro" />
-  <xacro:include filename="$(find archie_simulation)/robots/arche_mb/xacros/arche_mb_colors_gazebo.xacro" />
+  <xacro:include filename="$(find archie_simulation)/robots/archie_mb/xacros/archie_mb_gazebo.xacro" />
+  <xacro:include filename="$(find archie_simulation)/robots/archie_mb/xacros/archie_mb_colors_gazebo.xacro" />
   <!-- BODY -->
-  <xacro:include filename="$(find archie_simulation)/robots/arche_mb/xacros/arche_mb_body.xacro" />
+  <xacro:include filename="$(find archie_simulation)/robots/archie_mb/xacros/archie_mb_body.xacro" />
   <!-- WHEELS -->
-  <!-- <xacro:include filename="$(find archie_simulation)/robots/arche_mb/xacros/omni_wheel.xacro" /> -->
-  <xacro:include filename="$(find archie_simulation)/robots/arche_mb/xacros/mecanum_wheel.xacro" />
+  <!-- <xacro:include filename="$(find archie_simulation)/robots/archie_mb/xacros/omni_wheel.xacro" /> -->
+  <xacro:include filename="$(find archie_simulation)/robots/archie_mb/xacros/mecanum_wheel.xacro" />
   <!--DOCKING ADAPTER  -->
-  <xacro:include filename="$(find archie_simulation)/robots/arche_mb/xacros/docking_adapter.xacro" />
+  <xacro:include filename="$(find archie_simulation)/robots/archie_mb/xacros/docking_adapter.xacro" />
   <!-- SENSORS -->
-  <!-- <xacro:include filename="$(find archie_simulation)/robots/arche_mb/xacros/sick_S300.xacro" /> -->
+  <!-- <xacro:include filename="$(find archie_simulation)/robots/archie_mb/xacros/sick_S300.xacro" /> -->
   <!-- rplidar_a2 gazebo reference -->
-  <xacro:include filename="$(find archie_simulation)/robots/arche_mb/xacros/rplidar_a2.gazebo.xacro" />
+  <xacro:include filename="$(find archie_simulation)/robots/archie_mb/xacros/rplidar_a2.gazebo.xacro" />
   <!-- Microscan - Comment/Uncomment if required -->
-  <xacro:include filename="$(find archie_simulation)/robots/arche_mb/xacros/micro_scan.xacro" />
+  <xacro:include filename="$(find archie_simulation)/robots/archie_mb/xacros/micro_scan.xacro" />
   <!--Ultrasonics, cameras and IMU's  -->
   <!-- Depth Camera Realsense d435i-->
-  <xacro:include filename="$(find archie_simulation)/robots/arche_mb/xacros/depth_camera.xacro" />
+  <xacro:include filename="$(find archie_simulation)/robots/archie_mb/xacros/depth_camera.xacro" />
   <!-- Depth Camera ORBECC Astra (ONLY VISUAL)-->
-  <xacro:include filename="$(find archie_simulation)/robots/arche_mb/xacros/astra_rgbd_macro.xacro" />
+  <xacro:include filename="$(find archie_simulation)/robots/archie_mb/xacros/astra_rgbd_macro.xacro" />
   <!-->
-  <xacro:include filename="$(find archie_simulation)/robots/arche_mb/xacros/imu.xacro" />
-  <xacro:include filename="$(find archie_simulation)/robots/arche_mb/xacros/ultrasonic.xacro" />
+  <xacro:include filename="$(find archie_simulation)/robots/archie_mb/xacros/imu.xacro" />
+  <xacro:include filename="$(find archie_simulation)/robots/archie_mb/xacros/ultrasonic.xacro" />
   <-->
-  <!-- <xacro:include filename="$(find archie_simulation)/robots/arche_mb/xacros/camera.xacro" />  -->
+  <!-- <xacro:include filename="$(find archie_simulation)/robots/archie_mb/xacros/camera.xacro" />  -->
 <!-- ################################################################################## -->
     <!-- BASE-FOOTPRINT -->
@@ -52,9 +52,9 @@
     <!-- color="Yellow" z_offset="${chassis_center_to_base_footprint_z_offset}"> -->
   <!-- Base link macro -->
-  <xacro:arche_mb_base name="base_footprint" parent="base_link" lenght="${chassis_lenght}"
+  <xacro:archie_mb_base name="base_footprint" parent="base_link" lenght="${chassis_lenght}"
     width="${chassis_width}" height="${chassis_height}" mass="${chassis_weight}"
     color="Yellow" z_offset="${chassis_bottom_z_offset}">
     <joint_origin xyz="0 0 0" rpy="0 0 0" />
-  </xacro:arche_mb_base>
+  </xacro:archie_mb_base>
 <!-- **** ELECTRONICS BOX (MODULE) - height 100 mm ****  -->
 <!-- /batteries height is 76 mm whenlaying on the side. -->
@@ -150,21 +150,21 @@
     </xacro:shaft_link>
   <!-- Invoke Wheel Macros -->
-  <xacro:mecanum_wheel_152 name="arche_mb_mecanum_wheel_front_left" parent="base_footprint" diameter="${wheel_diameter}" width="${wheel_width}" mass="${wheel_weight}" color="White"
-      mesh_file_name="package://archie_simulation/robots/arche_mb/meshes/mecanum_wheel_left.STL" mesh_scale_x="${1*SCALE_mm_to_m}"
+  <xacro:mecanum_wheel_152 name="archie_mb_mecanum_wheel_front_left" parent="base_footprint" diameter="${wheel_diameter}" width="${wheel_width}" mass="${wheel_weight}" color="White"
+      mesh_file_name="package://archie_simulation/robots/archie_mb/meshes/mecanum_wheel_left.STL" mesh_scale_x="${1*SCALE_mm_to_m}"
       mesh_scale_y="${0.92*SCALE_mm_to_m}" mesh_scale_z="${1.52*SCALE_mm_to_m}">
     <origin xyz="${left_front_wheel_x_offset} ${left_front_wheel_y_offset+shaft_lenght} ${left_front_wheel_z_offset}" rpy="0 0 0" />
   </xacro:mecanum_wheel_152>
-  <xacro:mecanum_wheel_152 name="arche_mb_mecanum_wheel_front_right" parent="base_footprint" diameter="${wheel_diameter}" width="${wheel_width}" mass="${wheel_weight}" color="White"
-      mesh_file_name="package://archie_simulation/robots/arche_mb/meshes/mecanum_wheel_right.STL" mesh_scale_x="${1*SCALE_mm_to_m}"
+  <xacro:mecanum_wheel_152 name="archie_mb_mecanum_wheel_front_right" parent="base_footprint" diameter="${wheel_diameter}" width="${wheel_width}" mass="${wheel_weight}" color="White"
+      mesh_file_name="package://archie_simulation/robots/archie_mb/meshes/mecanum_wheel_right.STL" mesh_scale_x="${1*SCALE_mm_to_m}"
       mesh_scale_y="${0.92*SCALE_mm_to_m}" mesh_scale_z="${1.52*SCALE_mm_to_m}">
     <origin xyz="${left_front_wheel_x_offset} ${-(left_front_wheel_y_offset+shaft_lenght)} ${left_front_wheel_z_offset}" rpy="0 0 0" />
   </xacro:mecanum_wheel_152>
-  <xacro:mecanum_wheel_152 name="arche_mb_mecanum_wheel_back_left" parent="base_footprint" diameter="${wheel_diameter}" width="${wheel_width}" mass="${wheel_weight}" color="White"
-      mesh_file_name="package://archie_simulation/robots/arche_mb/meshes/mecanum_wheel_left.STL" mesh_scale_x="${1*SCALE_mm_to_m}"
+  <xacro:mecanum_wheel_152 name="archie_mb_mecanum_wheel_back_left" parent="base_footprint" diameter="${wheel_diameter}" width="${wheel_width}" mass="${wheel_weight}" color="White"
+      mesh_file_name="package://archie_simulation/robots/archie_mb/meshes/mecanum_wheel_left.STL" mesh_scale_x="${1*SCALE_mm_to_m}"
       mesh_scale_y="${0.92*SCALE_mm_to_m}" mesh_scale_z="${1.52*SCALE_mm_to_m}">
     <origin xyz="${-left_front_wheel_x_offset} ${left_front_wheel_y_offset+shaft_lenght} ${left_front_wheel_z_offset}" rpy="0 0 0" />
   </xacro:mecanum_wheel_152>
-  <xacro:mecanum_wheel_152 name="arche_mb_mecanum_wheel_back_right" parent="base_footprint" diameter="${wheel_diameter}" width="${wheel_width}" mass="${wheel_weight}" color="White"
-      mesh_file_name="package://archie_simulation/robots/arche_mb/meshes/mecanum_wheel_right.STL" mesh_scale_x="${1*SCALE_mm_to_m}"
+  <xacro:mecanum_wheel_152 name="archie_mb_mecanum_wheel_back_right" parent="base_footprint" diameter="${wheel_diameter}" width="${wheel_width}" mass="${wheel_weight}" color="White"
+      mesh_file_name="package://archie_simulation/robots/archie_mb/meshes/mecanum_wheel_right.STL" mesh_scale_x="${1*SCALE_mm_to_m}"
       mesh_scale_y="${0.92*SCALE_mm_to_m}" mesh_scale_z="${1.52*SCALE_mm_to_m}">
     <origin xyz="${-left_front_wheel_x_offset} ${-(left_front_wheel_y_offset+shaft_lenght)} ${left_front_wheel_z_offset}" rpy="0 0 0" />
@@ -202,5 +202,5 @@
       <origin xyz="0 0 -0.0308" rpy="1.5707 0 4.71"/> <!-- Move the mesh down on Z axis, as the joint is at the laser beam plane -->
       <geometry>
-        <mesh filename="package://archie_simulation/robots/arche_mb/meshes/rplidar.dae" scale="0.001 0.001 0.001" />
+        <mesh filename="package://archie_simulation/robots/archie_mb/meshes/rplidar.dae" scale="0.001 0.001 0.001" />
       </geometry>
     </collision>
@@ -208,5 +208,5 @@
       <origin xyz="0 0 -0.0308" rpy="1.5707 0 4.71"/>
       <geometry>
-        <mesh filename="package://archie_simulation/robots/arche_mb/meshes/rplidar.dae" scale="0.001 0.001 0.001" />
+        <mesh filename="package://archie_simulation/robots/archie_mb/meshes/rplidar.dae" scale="0.001 0.001 0.001" />
       </geometry>
     </visual>
@@ -308,37 +308,37 @@
   </xacro:depth_camera>
   <!-- TRANSMISSIONS -->
-  <transmission name="arche_mb_mecanum_wheel_front_left">
+  <transmission name="archie_mb_mecanum_wheel_front_left">
     <type>transmission_interface/SimpleTransmission</type>
-    <joint name="arche_mb_mecanum_wheel_front_left_joint">
+    <joint name="archie_mb_mecanum_wheel_front_left_joint">
       <hardwareInterface>hardware_interface/VelocityJointInterface</hardwareInterface>
     </joint>
-    <actuator name="arche_mb_mecanum_wheel_front_left_motor">
+    <actuator name="archie_mb_mecanum_wheel_front_left_motor">
       <mechanicalReduction>1</mechanicalReduction>
     </actuator>
   </transmission>
-  <transmission name="arche_mb_mecanum_wheel_front_right">
+  <transmission name="archie_mb_mecanum_wheel_front_right">
     <type>transmission_interface/SimpleTransmission</type>
-    <joint name="arche_mb_mecanum_wheel_front_right_joint">
+    <joint name="archie_mb_mecanum_wheel_front_right_joint">
       <hardwareInterface>hardware_interface/VelocityJointInterface</hardwareInterface>
     </joint>
-    <actuator name="arche_mb_mecanum_wheel_front_right_motor">
+    <actuator name="archie_mb_mecanum_wheel_front_right_motor">
       <mechanicalReduction>1</mechanicalReduction>
     </actuator>
   </transmission>
-  <transmission name="arche_mb_mecanum_wheel_back_left">
+  <transmission name="archie_mb_mecanum_wheel_back_left">
     <type>transmission_interface/SimpleTransmission</type>
-    <joint name="arche_mb_mecanum_wheel_back_left_joint">
+    <joint name="archie_mb_mecanum_wheel_back_left_joint">
       <hardwareInterface>hardware_interface/VelocityJointInterface</hardwareInterface>
     </joint>
-    <actuator name="arche_mb_mecanum_wheel_back_left_motor">
+    <actuator name="archie_mb_mecanum_wheel_back_left_motor">
       <mechanicalReduction>1</mechanicalReduction>
     </actuator>
   </transmission>
-  <transmission name="arche_mb_mecanum_wheel_back_right">
+  <transmission name="archie_mb_mecanum_wheel_back_right">
     <type>transmission_interface/SimpleTransmission</type>
-    <joint name="arche_mb_mecanum_wheel_back_right_joint">
+    <joint name="archie_mb_mecanum_wheel_back_right_joint">
       <hardwareInterface>hardware_interface/VelocityJointInterface</hardwareInterface>
     </joint>
-    <actuator name="arche_mb_mecanum_wheel_back_right_motor">
+    <actuator name="archie_mb_mecanum_wheel_back_right_motor">
       <mechanicalReduction>1</mechanicalReduction>
     </actuator>

File: robots/archie_mb/xacros/archie_mb_body.xacro (robot description, xacro)
@@ -1,5 +1,5 @@
 <?xml version="1.0"?>
-<robot xmlns:xacro="http://www.ros.org/wiki/xacro" name="arche_mb">
-  <xacro:macro name="arche_mb_base" params="name parent *joint_origin lenght width height mass color z_offset">
+<robot xmlns:xacro="http://www.ros.org/wiki/xacro" name="archie_mb">
+  <xacro:macro name="archie_mb_base" params="name parent *joint_origin lenght width height mass color z_offset">
     <joint name="${name}_joint" type="fixed">
       <xacro:insert_block name="joint_origin" />
@@ -17,5 +17,5 @@
           <geometry>
             <box size="${lenght} ${width} ${height}"/>
-            <!-- <mesh filename="package://archie_simulation/robots/arche_mb/meshes/arche_mb_full_body.STL" scale="0.01 0.01 0.01"/> -->
+            <!-- <mesh filename="package://archie_simulation/robots/archie_mb/meshes/archie_mb_full_body.STL" scale="0.01 0.01 0.01"/> -->
           </geometry>
         <material name="${color}" />
@@ -26,5 +26,5 @@
         <geometry>
             <box size="${lenght} ${width} ${height}"/>
-           <!-- <mesh filename="package://archie_simulation/robots/arche_mb/meshes/MPO-500-BODY.dae" scale="0.001 0.001 0.001"/> -->
+           <!-- <mesh filename="package://archie_simulation/robots/archie_mb/meshes/MPO-500-BODY.dae" scale="0.001 0.001 0.001"/> -->
         </geometry>
       </collision>
@@ -60,5 +60,5 @@
           <origin xyz="0 0 ${height/2}" rpy="0 0 0" />
           <geometry>
-            <!-- <mesh filename="package://archie_simulation/robots/arche_mb/meshes/archie_electronics_link.STL" scale="0.001 0.001 0.001"/> -->
+            <!-- <mesh filename="package://archie_simulation/robots/archie_mb/meshes/archie_electronics_link.STL" scale="0.001 0.001 0.001"/> -->
             <box size="${lenght} ${width} ${height}"/>
           </geometry>

File: robots/archie_mb/xacros/archie_mb_colors_gazebo.xacro (robot description, xacro)
@@ -1,3 +1,3 @@
 <?xml version="1.0"?>
-<robot name="arche_mb" xmlns:xacro="http://www.ros.org/wiki/xacro">
+<robot name="archie_mb" xmlns:xacro="http://www.ros.org/wiki/xacro">
 </robot>

File: robots/archie_mb/xacros/archie_mb_gazebo.xacro (robot description, xacro)
@@ -1,4 +1,4 @@
 <?xml version="1.0"?>
-<robot name="arche_mb" xmlns:xacro="http://www.ros.org/wiki/xacro">
+<robot name="archie_mb" xmlns:xacro="http://www.ros.org/wiki/xacro">
   <!-- All static links get collapsed down to base_link in Gazebo, so that's
        the one to apply the colour to (in Gazebo 5+). -->
@@ -55,14 +55,14 @@
 <!-- !######### WHEELS - Gazebo  mu1, mu2 and material are defined in
      ! mecanum_wheel.xacro -->
-  <!-- <gazebo reference="arche_mb_mecanum_wheel_front_left_link">
+  <!-- <gazebo reference="archie_mb_mecanum_wheel_front_left_link">
     <material>Gazebo/Grey</material>
   </gazebo>
-  <gazebo reference="arche_mb_mecanum_wheel_back_left_link">
+  <gazebo reference="archie_mb_mecanum_wheel_back_left_link">
     <material>Gazebo/Grey</material>
   </gazebo>
-  <gazebo reference="arche_mb_mecanum_wheel_front_right_link">
+  <gazebo reference="archie_mb_mecanum_wheel_front_right_link">
     <material>Gazebo/Grey</material>
   </gazebo>
-  <gazebo reference="arche_mb_mecanum_wheel_back_right_link">
+  <gazebo reference="archie_mb_mecanum_wheel_back_right_link">
     <material>Gazebo/Grey</material>
   </gazebo> -->
@@ -296,5 +296,5 @@
 </gazebo>
 <gazebo>
-    <plugin name="arche_mb_controller" filename="libgazebo_ros_planar_move.so">
+    <plugin name="archie_mb_controller" filename="libgazebo_ros_planar_move.so">
       <commandTopic>cmd_vel</commandTopic>
       <odometryTopic>odom</odometryTopic>

File: robots/archie_mb/xacros/astra_rgbd_macro.xacro (robot description, xacro)
@@ -1,4 +1,4 @@
 <?xml version="1.0"?>
-<robot xmlns:xacro="http://www.ros.org/wiki/xacro" name="arche_mb">
+<robot xmlns:xacro="http://www.ros.org/wiki/xacro" name="archie_mb">
 <xacro:macro name="astra_depth_camera" params="name">
 <!-- **** ORBBEC ASTRA RGBD CAMERA  ****  -->
@@ -21,7 +21,7 @@
       <origin xyz="-0.01 0 -0.03" rpy="1.5707 0 1.5707"/>
       <geometry>
-        <mesh filename="package://archie_simulation/robots/arche_mb/meshes/astra.dae" scale="0.001 0.001 0.001" />
-		<!-- <mesh filename="package://archie_simulation/robots/arche_mb/meshes/realsense_d435.dae"/> -->
-		<!-- <mesh filename="package://archie_simulation/robots/arche_mb/meshes/IntelRealsense_D435_Multibody.stl" scale="0.001 0.001 0.001"/> -->
+        <mesh filename="package://archie_simulation/robots/archie_mb/meshes/astra.dae" scale="0.001 0.001 0.001" />
+		<!-- <mesh filename="package://archie_simulation/robots/archie_mb/meshes/realsense_d435.dae"/> -->
+		<!-- <mesh filename="package://archie_simulation/robots/archie_mb/meshes/IntelRealsense_D435_Multibody.stl" scale="0.001 0.001 0.001"/> -->
       </geometry>
     </visual>

File: robots/archie_mb/xacros/depth_camera.xacro (robot description, xacro)
@@ -1,4 +1,4 @@
 <?xml version="1.0"?>
-<robot xmlns:xacro="http://www.ros.org/wiki/xacro" name="arche_mb">
+<robot xmlns:xacro="http://www.ros.org/wiki/xacro" name="archie_mb">
 	<xacro:macro name="depth_camera" params="name parent *origin">
 	  	<xacro:property name="depth_camera_link" value="0.05" />
@@ -29,5 +29,5 @@
 			      <origin xyz="0 -0.0175 0" rpy="1.570796 0 1.570796"/>
 			      <geometry>
-			      	<mesh filename="package://archie_simulation/robots/arche_mb/meshes/realsense_d435.dae"/>
+			      	<mesh filename="package://archie_simulation/robots/archie_mb/meshes/realsense_d435.dae"/>
 			      </geometry>
 			      <material name="Red">

File: robots/archie_mb/xacros/docking_adapter.xacro (robot description, xacro)
@@ -1,4 +1,4 @@
 <?xml version="1.0"?>
-<robot xmlns:xacro="http://www.ros.org/wiki/xacro" name="arche_mb">
+<robot xmlns:xacro="http://www.ros.org/wiki/xacro" name="archie_mb">
   <xacro:macro name="docking_adapter" params="name parent *origin">
     <joint name="${name}_joint" type="fixed">
@@ -17,5 +17,5 @@
         <origin xyz="0 0 0.0" rpy="0 0 0" />
       <geometry>
-        <mesh filename="package://archie_simulation/robots/arche_mb/meshes/arche_mb_charge_port.dae" scale="0.1 0.1 0.1" />
+        <mesh filename="package://archie_simulation/robots/archie_mb/meshes/archie_mb_charge_port.dae" scale="0.1 0.1 0.1" />
         </geometry>
       </visual>
@@ -23,5 +23,5 @@
         <origin xyz="0 0 0.0" rpy="0 0 0" />
         <geometry>
-          <mesh filename="package://archie_simulation/robots/arche_mb/meshes/arche_mb_charge_port.dae" scale="0.1 0.1 0.1" />
+          <mesh filename="package://archie_simulation/robots/archie_mb/meshes/archie_mb_charge_port.dae" scale="0.1 0.1 0.1" />
         </geometry>
       </collision>

File: robots/archie_mb/xacros/materials.xacro (robot description, xacro)
@@ -1,5 +1,5 @@
 <?xml version="1.0"?>
 <robot xmlns:xacro="http://www.ros.org/wiki/xacro" name="materials">
-<!-- Properties file for arche_mb robot -->
+<!-- Properties file for archie_mb robot -->
 <!-- Created by Stefan -->
 <!-- IICT-BAS BG - Version 1.0 from Feb. 15-th, 2021. -->

File: robots/archie_mb/xacros/mecanum_wheel.xacro (robot description, xacro)
@@ -1,4 +1,4 @@
 <?xml version="1.0"?>
-<robot xmlns:xacro="http://www.ros.org/wiki/xacro" name="arche_mb">
+<robot xmlns:xacro="http://www.ros.org/wiki/xacro" name="archie_mb">
   <xacro:macro name="shaft_joint" params="name *origin">
   <joint name="${name}_wheel_shaft_joint" type="fixed">
@@ -58,5 +58,5 @@
      <geometry>
         <!-- <mesh filename="package://archie_simulation/robots/mpo_500/meshes/MPO-500-WHEEL.dae" scale="0.001 0.001 0.001"/> -->
-        <!-- <mesh filename="package://archie_simulation/robots/arche_mb/meshes/mecanum_wheel_left.STL" scale="0.001 0.001 0.001"/> -->
+        <!-- <mesh filename="package://archie_simulation/robots/archie_mb/meshes/mecanum_wheel_left.STL" scale="0.001 0.001 0.001"/> -->
         <mesh filename="${mesh_file_name}" scale="${mesh_scale_x} ${mesh_scale_y} ${mesh_scale_z}"/>
       <!-- <cylinder radius="0.076" length="0.046"/> -->

File: robots/archie_mb/xacros/omni_wheel.xacro (robot description, xacro)
@@ -1,4 +1,4 @@
 <?xml version="1.0"?>
-<robot xmlns:xacro="http://www.ros.org/wiki/xacro" name="arche_mb">
+<robot xmlns:xacro="http://www.ros.org/wiki/xacro" name="archie_mb">
   <xacro:macro name="omni_wheel_250" params="name parent *origin">
    <joint name="${name}_joint" type="revolute">
@@ -22,5 +22,5 @@
      <origin xyz="0 0 0" rpy="0 0 0"/>
      <geometry>
-        <mesh filename="package://archie_simulation/robots/arche_mb/meshes/MPO-500-WHEEL.dae" scale="0.001 0.001 0.001"/>
+        <mesh filename="package://archie_simulation/robots/archie_mb/meshes/MPO-500-WHEEL.dae" scale="0.001 0.001 0.001"/>
      </geometry>
     </visual>
@@ -28,5 +28,5 @@
      <origin xyz="0 0 0" rpy="0 1.57 1.57" />
      <geometry>
-        <!-- <mesh filename="package://archie_simulation/robots/arche_mb/meshes/MPO-500-WHEEL.dae" scale="0.001 0.001 0.001"/> -->
+        <!-- <mesh filename="package://archie_simulation/robots/archie_mb/meshes/MPO-500-WHEEL.dae" scale="0.001 0.001 0.001"/> -->
        <!-- <cylinder radius="0.126" length="0.110"/> -->
       <sphere radius="0.117" />

File: robots/archie_mb/xacros/properties.xacro (robot description, xacro)
@@ -1,5 +1,5 @@
 <?xml version="1.0"?>
 <robot xmlns:xacro="http://www.ros.org/wiki/xacro" name="properties">
-<!-- Properties file for arche_mb robot -->
+<!-- Properties file for archie_mb robot -->
 <!-- Created by Stefan -->
 <!-- IICT-BAS BG - Version 1.0 from Feb. 15-th, 2021. -->

File: robots/archie_mb/xacros/rplidar_a2.gazebo.xacro (robot description, xacro)
@@ -1,4 +1,4 @@
 <?xml version="1.0"?>
-<robot name="arche_mb" xmlns:xacro="http://www.ros.org/wiki/xacro">
+<robot name="archie_mb" xmlns:xacro="http://www.ros.org/wiki/xacro">
   <!-- If you cant't use your GPU comment RpLidar using GPU and uncomment RpLidar using CPU
     gazebo plugin. -->

File: robots/archie_mb/xacros/rplidar_a2.macro.xacro (robot description, xacro)
@@ -1,4 +1,4 @@
 <?xml version="1.0"?>
-<robot name="arche_mb" xmlns:xacro="http://www.ros.org/wiki/xacro">
+<robot name="archie_mb" xmlns:xacro="http://www.ros.org/wiki/xacro">
   <!-- <joint name="rplidar_joint" type="fixed">
     <axis xyz="0 1 0" />
