Commit message: Correct typo arche_mb to archie_mb in all files

File: robots/archie_mb/xacros/sick_laser.xacro (robot description, xacro)
@@ -1,4 +1,4 @@
 <?xml version="1.0"?>
-<robot xmlns:xacro="http://www.ros.org/wiki/xacro" name="arche_mb">
+<robot xmlns:xacro="http://www.ros.org/wiki/xacro" name="archie_mb">
   <xacro:macro name="sick_laser_v0" params="name parent *origin ros_topic">
     <joint name="${name}_joint" type="fixed">
@@ -18,5 +18,5 @@
       <origin xyz="0 0 -0.12" rpy="-1.57 0 3.14" />
         <geometry>
-        <mesh filename="package://archie_simulation/robots/arche_mb/meshes/SICK-S300.dae" scale="0.001 0.001 0.001" />
+        <mesh filename="package://archie_simulation/robots/archie_mb/meshes/SICK-S300.dae" scale="0.001 0.001 0.001" />
         </geometry>
       </visual>
@@ -24,5 +24,5 @@
         <origin xyz="0 0 0" rpy="-1.57 0 3.14" />
         <geometry>
-        <mesh filename="package://archie_simulation/robots/arche_mb/meshes/SICK-S300.dae" scale="0.001 0.001 0.001" />
+        <mesh filename="package://archie_simulation/robots/archie_mb/meshes/SICK-S300.dae" scale="0.001 0.001 0.001" />
         </geometry>
       </collision>
@@ -30,5 +30,5 @@
 <!--  <origin xyz="-0.0 0 -0.06" rpy="1.57 0 0" />
       <geometry>
-      <mesh filename="package://archie_simulation/robots/arche_mb/meshes/SICK-MICROSCAN3.dae" scale="0.001 0.001 0.001" />
+      <mesh filename="package://archie_simulation/robots/archie_mb/meshes/SICK-MICROSCAN3.dae" scale="0.001 0.001 0.001" />
       </geometry>
       </visual>
